File: rpi_pico_flexypin/rpi_pico_flexypin.kicad_sch (KiCad schematic)
At the start: 8 parts, among them J1 Conn_01x20, J2 Conn_01x03, J3 Conn_01x20, J4 Conn_01x17, J5 Conn_01x17, J6 Conn_Debug, SW1 SW_RST, U1 RaspberryPi_Pico

Commit message: Change Pico Adapters' Reset Button to SMD
Parts:
- SW1: footprint Button_Switch_THT:SW_PUSH_6mm -> Button_Switch_SMD:SW_Push_1P1T_NO_6x6mm_H9.5mm
