File: rpi_pico_uno_flexypin/rpi_pico_uno_flexypin.kicad_sch (KiCad schematic)
At the start: 11 parts, among them J1 Conn_01x20, J2 Conn_01x03, J3 Conn_01x20, J4 Conn_01x03, J5 Conn_SPI, J6 Conn_01x08, J7 Conn_01x06, J8 Conn_01x10, J9 Conn_01x08, SW1 SW_RST, U1 RaspberryPi_Pico

Commit message: Change Pico Adapters' Reset Button to SMD
Parts:
- SW1: footprint Button_Switch_THT:SW_PUSH_6mm -> Button_Switch_SMD:SW_Push_1P1T_NO_6x6mm_H9.5mm
Changed lines of the file:
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@@
     (property "Reference" "SW1" (id 0) (at 153.67 41.91 0))
     (property "Value" "SW_RST" (id 1) (at 153.67 46.99 0))
-    (property "Footprint" "Button_Switch_THT:SW_PUSH_6mm" (id 2) (at 153.67 44.45 0)
+    (property "Footprint" "Button_Switch_SMD:SW_Push_1P1T_NO_6x6mm_H9.5mm" (id 2) (at 153.67 44.45 0)
       (effects (font (size 1.27 1.27)) hide)
     )
@@
     )
     (path "/9ada2fb0-6951-4068-9e43-302e463cabaa"
-      (reference "SW1") (unit 1) (value "SW_RST") (footprint "Button_Switch_THT:SW_PUSH_6mm")
+      (reference "SW1") (unit 1) (value "SW_RST") (footprint "Button_Switch_SMD:SW_Push_1P1T_NO_6x6mm_H9.5mm")
     )
     (path "/66e6c744-b8b4-45a4-a3cc-59a8b83b0a84"
